File: pcb/BlinkyTile_controller.brd (EAGLE design)
At the start: 49.8 x 47.4 mm, 9 parts

Commit message: Rev E of pcb, control pcb
Parts:
- added C2: .1uF, adafruit:C0603
- added SW1, SW2: SPST_TACT-EVQQ2, adafruit:EVQ-Q2
- added U1: Tiny85-20-SMT, SparkFun-DigitalIC:SO08-EIAJ
Connections:
- new net N$3: SW1.B', SW2.B, U1.1
- net 5V: now also C2.1, U1.8; no longer U$2.PWRVIA1, U$2.PWRVIA2, U$2.PWRVIA3, U$2.PWRVIA4, U$2.PWRVIA5, U$2.PWRVIA6, U$3.PWRVIA1, U$3.PWRVIA2, U$3.PWRVIA3, U$3.PWRVIA4, U$3.PWRVIA5, U$3.PWRVIA6, U$4.PWRVIA1, U$4.PWRVIA2, U$4.PWRVIA3, U$4.PWRVIA4, U$4.PWRVIA5, U$4.PWRVIA6, U$5.PWRVIA1, U$5.PWRVIA2, U$5.PWRVIA3, U$5.PWRVIA4, U$5.PWRVIA5, U$5.PWRVIA6, U$6.PWRVIA1, U$6.PWRVIA2, U$6.PWRVIA3, U$6.PWRVIA4, U$6.PWRVIA5, U$6.PWRVIA6
- net DATA: now also U1.6; no longer U$2.SIGVIA1, U$2.SIGVIA2, U$2.SIGVIA3, U$3.SIGVIA1, U$3.SIGVIA2, U$3.SIGVIA3, U$4.SIGVIA1, U$4.SIGVIA2, U$4.SIGVIA3, U$5.SIGVIA1, U$5.SIGVIA2, U$5.SIGVIA3, U$6.SIGVIA1, U$6.SIGVIA2, U$6.SIGVIA3
- net GND: now also C2.2, SW1.A, SW2.A', U1.4; no longer U$2.GNDVIA1, U$2.GNDVIA2, U$2.GNDVIA3, U$2.GNDVIA4, U$2.GNDVIA5, U$2.GNDVIA6, U$3.GNDVIA1, U$3.GNDVIA2, U$3.GNDVIA3, U$3.GNDVIA4, U$3.GNDVIA5, U$3.GNDVIA6, U$4.GNDVIA1, U$4.GNDVIA2, U$4.GNDVIA3, U$4.GNDVIA4, U$4.GNDVIA5, U$4.GNDVIA6, U$5.GNDVIA1, U$5.GNDVIA2, U$5.GNDVIA3, U$5.GNDVIA4, U$5.GNDVIA5, U$5.GNDVIA6, U$6.GNDVIA1, U$6.GNDVIA2, U$6.GNDVIA3, U$6.GNDVIA4, U$6.GNDVIA5, U$6.GNDVIA6
Routing:
- net GND: track 123.6 -> 145.1 mm, vias 18 -> 23
- net N$3: track 0.00 -> 11.5 mm, vias 0 -> 1
- net DATA: track 11.7 -> 21.9 mm
- net 5V: track 3.07 -> 7.60 mm, vias 2 -> 3
Other:
- board text added: "BlinkyTile Rev. D"
- board text removed: "BlinkyTile Rev. E"
