File: pcb/BlinkyTile_panel.brd (EAGLE design)
At the start: 260 x 187.7 mm, 144 parts

Commit message: Add RevF panel design, as submitted
Parts:
- removed C3, C4: .1uF, adafruit:C0603
- removed R5, R7: 75, adafruit:R0603
- removed R6, R8: 10k, adafruit:R0603
- removed U$13, U$14, U$15, U$16, U$17, U$19, U$20, U$21, U$22, U$23: D_EDGESLOT, dodocohedreled:D_EDGE_SLOT
- removed U$18, U$24: WS2822S_LED, blinkinlabs:WS2822S_LED
- added E$1, E$10, E$100, E$101, E$102, E$103, E$104, E$105, E$106, E$107, E$108, E$109, E$11, E$110, E$111, E$112, E$113, E$114, E$115, E$116, E$117, E$118, E$119, E$12, E$120, E$121, E$122, E$123, E$124, E$125, E$126, E$127, E$128, E$129, E$13, E$130, E$131, E$132, E$133, E$134, E$135, E$136, E$137, E$138, E$139, E$14, E$140, E$141, E$142, E$143, E$144, E$145, E$146, E$147, E$148, E$149, E$15, E$150, E$151, E$152, E$16, E$17, E$18, E$19, E$2, E$20, E$21, E$22, E$33, E$34, E$35, E$36, E$37, E$38, E$39, E$40, E$41, E$42, E$43, E$44, E$45, E$46, E$47, E$48, E$49, E$5, E$50, E$51, E$52, E$53, E$54, E$55, E$56, E$57, E$58, E$59, E$6, E$60, E$61, E$62, E$63, E$64, E$65, E$66, E$67, E$68, E$69, E$7, E$70, E$71, E$72, E$73, E$74, E$75, E$76, E$77, E$78, E$79, E$8, E$80, E$81, E$82, E$83, E$84, E$85, E$86, E$87, E$88, E$89, E$9, E$90, E$91, E$92, E$93, E$94, E$95, E$96, E$97, E$98, E$99: (no value), dodocohedreled:MOUSE_BITE
- U$1, U$10, U$11, U$2, U$25, U$26, U$27, U$28, U$29, U$3, U$31, U$32, U$33, U$34, U$35, U$37, U$38, U$39, U$4, U$40, U$41, U$43, U$44, U$45, U$46, U$47, U$49, U$5, U$50, U$51, U$52, U$53, U$55, U$56, U$57, U$58, U$59, U$6, U$61, U$62, U$63, U$64, U$65, U$67, U$68, U$69, U$70, U$71, U$73, U$74, U$75, U$76, U$77, U$79, U$8, U$80, U$81, U$82, U$83, U$85, U$86, U$87, U$88, U$89, U$9, U$91, U$92, U$93, U$94, U$95: value D_EDGESLOT -> D_EDGEMOD; device dodocohedreled:D_EDGE_SLOT -> dodocohedreled:D_EDGE_SLOT_MOD
- moved U$65 214.1 mm to (170.5, -61.4), turned to 36 degrees
- moved U$63 190.9 mm to (178.3, -37.7), turned to 108 degrees
- moved U$64 187.5 mm to (145.6, -61.4), turned to 324 degrees
- moved R17 185.1 mm to (158.2, 5.40)
- moved U$76 184.2 mm to (40.1, -61.3), turned to 324 degrees
- moved R21 184.1 mm to (158.1, -49.6), turned to 90 degrees
- moved R18 183.8 mm to (159.8, 5.40)
- moved C11 182.5 mm to (159.7, -49.6), turned to 270 degrees
- moved U$50 182.0 mm to (178.4, -6.50)
- moved U$53 182.0 mm to (145.8, 17.2)
- moved U$49 182.0 mm to (158.2, -21.2)
- moved U$51 182.0 mm to (138.0, -6.50)
- moved U$52 182.0 mm to (170.7, 17.2)
- moved U$54 182.0 mm to (158.2, 0.00)
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Connections:
- removed net 5V2: R5.1, U$13.P$2, U$13.P$4, U$13.P$7, U$13.P$9, U$14.P$2, U$14.P$4, U$14.P$7, U$14.P$9, U$15.P$2, U$15.P$4, U$15.P$7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
- removed net 5V3: R7.1, U$19.P$2, U$19.P$4, U$19.P$7, U$19.P$9, U$20.P$2, U$20.P$4, U$20.P$7, U$20.P$9, U$21.P$2, U$21.P$4, U$21.P$7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
- removed net ADRI2: U$18.2
- removed net ADRI3: U$24.2
- removed net DATA2: R6.2, U$13.P$3, U$13.P$8, U$14.P$3, U$14.P$8, U$15.P$3, U$15.P$8, U$16.P$3, U$16.P$8, U$17.P$3, U$17.P$8
- removed net DATA3: R8.2, U$19.P$3, U$19.P$8, U$20.P$3, U$20.P$8, U$21.P$3, U$21.P$8, U$22.P$3, U$22.P$8, U$23.P$3, U$23.P$8
- removed net GND2: C3.2, U$13.P$1, U$13.P$10, U$13.P$5, U$13.P$6, U$14.P$1, U$14.P$10, U$14.P$5, U$14.P$6, U$15.P$1, U$15.P$10, U$15.P$5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
- removed net GND3: C4.2, U$19.P$1, U$19.P$10, U$19.P$5, U$19.P$6, U$20.P$1, U$20.P$10, U$20.P$5, U$20.P$6, U$21.P$1, U$21.P$10, U$21.P$5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
- removed net N$11: C4.1, R7.2, U$24.3
- removed net N$12: R8.1, U$24.1
- removed net N$8: C3.1, R5.2, U$18.3
- removed net N$9: R6.1, U$18.1
- net 5V: now also U$2.PWRVIA1, U$2.PWRVIA3, U$2.PWRVIA4, U$2.PWRVIA6, U$3.PWRVIA1, U$3.PWRVIA3, U$3.PWRVIA4, U$3.PWRVIA6, U$4.PWRVIA1, U$4.PWRVIA3, U$4.PWRVIA4, U$4.PWRVIA6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
- net 5V1: now also U$1.PWRVIA1, U$1.PWRVIA3, U$1.PWRVIA4, U$1.PWRVIA6, U$10.PWRVIA1, U$10.PWRVIA3, U$10.PWRVIA4, U$10.PWRVIA6, U$11.PWRVIA1, U$11.PWRVIA3, U$11.PWRVIA4, U$11.PWRVIA6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
- net 5V10: now also U$61.PWRVIA1, U$61.PWRVIA3, U$61.PWRVIA4, U$61.PWRVIA6, U$62.PWRVIA1, U$62.PWRVIA3, U$62.PWRVIA4, U$62.PWRVIA6, U$63.PWRVIA1, U$63.PWRVIA3, U$63.PWRVIA4, U$63.PWRVIA6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
- net 5V11: now also U$67.PWRVIA1, U$67.PWRVIA3, U$67.PWRVIA4, U$67.PWRVIA6, U$68.PWRVIA1, U$68.PWRVIA3, U$68.PWRVIA4, U$68.PWRVIA6, U$69.PWRVIA1, U$69.PWRVIA3, U$69.PWRVIA4, U$69.PWRVIA6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
- net 5V12: now also U$73.PWRVIA1, U$73.PWRVIA3, U$73.PWRVIA4, U$73.PWRVIA6, U$74.PWRVIA1, U$74.PWRVIA3, U$74.PWRVIA4, U$74.PWRVIA6, U$75.PWRVIA1, U$75.PWRVIA3, U$75.PWRVIA4, U$75.PWRVIA6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
- net 5V13: now also U$79.PWRVIA1, U$79.PWRVIA3, U$79.PWRVIA4, U$79.PWRVIA6, U$80.PWRVIA1, U$80.PWRVIA3, U$80.PWRVIA4, U$80.PWRVIA6, U$81.PWRVIA1, U$81.PWRVIA3, U$81.PWRVIA4, U$81.PWRVIA6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
- net 5V14: now also U$85.PWRVIA1, U$85.PWRVIA3, U$85.PWRVIA4, U$85.PWRVIA6, U$86.PWRVIA1, U$86.PWRVIA3, U$86.PWRVIA4, U$86.PWRVIA6, U$87.PWRVIA1, U$87.PWRVIA3, U$87.PWRVIA4, U$87.PWRVIA6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
- net 5V15: now also U$91.PWRVIA1, U$91.PWRVIA3, U$91.PWRVIA4, U$91.PWRVIA6, U$92.PWRVIA1, U$92.PWRVIA3, U$92.PWRVIA4, U$92.PWRVIA6, U$93.PWRVIA1, U$93.PWRVIA3, U$93.PWRVIA4, U$93.PWRVIA6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
- net 5V4: now also U$25.PWRVIA1, U$25.PWRVIA3, U$25.PWRVIA4, U$25.PWRVIA6, U$26.PWRVIA1, U$26.PWRVIA3, U$26.PWRVIA4, U$26.PWRVIA6, U$27.PWRVIA1, U$27.PWRVIA3, U$27.PWRVIA4, U$27.PWRVIA6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
- net 5V5: now also U$31.PWRVIA1, U$31.PWRVIA3, U$31.PWRVIA4, U$31.PWRVIA6, U$32.PWRVIA1, U$32.PWRVIA3, U$32.PWRVIA4, U$32.PWRVIA6, U$33.PWRVIA1, U$33.PWRVIA3, U$33.PWRVIA4, U$33.PWRVIA6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
- net 5V6: now also U$37.PWRVIA1, U$37.PWRVIA3, U$37.PWRVIA4, U$37.PWRVIA6, U$38.PWRVIA1, U$38.PWRVIA3, U$38.PWRVIA4, U$38.PWRVIA6, U$39.PWRVIA1, U$39.PWRVIA3, U$39.PWRVIA4, U$39.PWRVIA6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
- net 5V7: now also U$43.PWRVIA1, U$43.PWRVIA3, U$43.PWRVIA4, U$43.PWRVIA6, U$44.PWRVIA1, U$44.PWRVIA3, U$44.PWRVIA4, U$44.PWRVIA6, U$45.PWRVIA1, U$45.PWRVIA3, U$45.PWRVIA4, U$45.PWRVIA6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
- net 5V8: now also U$49.PWRVIA1, U$49.PWRVIA3, U$49.PWRVIA4, U$49.PWRVIA6, U$50.PWRVIA1, U$50.PWRVIA3, U$50.PWRVIA4, U$50.PWRVIA6, U$51.PWRVIA1, U$51.PWRVIA3, U$51.PWRVIA4, U$51.PWRVIA6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
- net 5V9: now also U$55.PWRVIA1, U$55.PWRVIA3, U$55.PWRVIA4, U$55.PWRVIA6, U$56.PWRVIA1, U$56.PWRVIA3, U$56.PWRVIA4, U$56.PWRVIA6, U$57.PWRVIA1, U$57.PWRVIA3, U$57.PWRVIA4, U$57.PWRVIA6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
- net DATA: now also U$2.SIGVIA1, U$2.SIGVIA3, U$3.SIGVIA1, U$3.SIGVIA3, U$4.SIGVIA1, U$4.SIGVIA3, U$5.SIGVIA1, U$5.SIGVIA3, U$6.SIGVIA1, U$6.SIGVIA3
- net DATA1: now also U$1.SIGVIA1, U$1.SIGVIA3, U$10.SIGVIA1, U$10.SIGVIA3, U$11.SIGVIA1, U$11.SIGVIA3, U$8.SIGVIA1, U$8.SIGVIA3, U$9.SIGVIA1, U$9.SIGVIA3
- net DATA10: now also U$61.SIGVIA1, U$61.SIGVIA3, U$62.SIGVIA1, U$62.SIGVIA3, U$63.SIGVIA1, U$63.SIGVIA3, U$64.SIGVIA1, U$64.SIGVIA3, U$65.SIGVIA1, U$65.SIGVIA3
- net DATA11: now also U$67.SIGVIA1, U$67.SIGVIA3, U$68.SIGVIA1, U$68.SIGVIA3, U$69.SIGVIA1, U$69.SIGVIA3, U$70.SIGVIA1, U$70.SIGVIA3, U$71.SIGVIA1, U$71.SIGVIA3
- net DATA12: now also U$73.SIGVIA1, U$73.SIGVIA3, U$74.SIGVIA1, U$74.SIGVIA3, U$75.SIGVIA1, U$75.SIGVIA3, U$76.SIGVIA1, U$76.SIGVIA3, U$77.SIGVIA1, U$77.SIGVIA3
- net DATA13: now also U$79.SIGVIA1, U$79.SIGVIA3, U$80.SIGVIA1, U$80.SIGVIA3, U$81.SIGVIA1, U$81.SIGVIA3, U$82.SIGVIA1, U$82.SIGVIA3, U$83.SIGVIA1, U$83.SIGVIA3
- net DATA14: now also U$85.SIGVIA1, U$85.SIGVIA3, U$86.SIGVIA1, U$86.SIGVIA3, U$87.SIGVIA1, U$87.SIGVIA3, U$88.SIGVIA1, U$88.SIGVIA3, U$89.SIGVIA1, U$89.SIGVIA3
- net DATA15: now also U$91.SIGVIA1, U$91.SIGVIA3, U$92.SIGVIA1, U$92.SIGVIA3, U$93.SIGVIA1, U$93.SIGVIA3, U$94.SIGVIA1, U$94.SIGVIA3, U$95.SIGVIA1, U$95.SIGVIA3
- net DATA4: now also U$25.SIGVIA1, U$25.SIGVIA3, U$26.SIGVIA1, U$26.SIGVIA3, U$27.SIGVIA1, U$27.SIGVIA3, U$28.SIGVIA1, U$28.SIGVIA3, U$29.SIGVIA1, U$29.SIGVIA3
- net DATA5: now also U$31.SIGVIA1, U$31.SIGVIA3, U$32.SIGVIA1, U$32.SIGVIA3, U$33.SIGVIA1, U$33.SIGVIA3, U$34.SIGVIA1, U$34.SIGVIA3, U$35.SIGVIA1, U$35.SIGVIA3
- net DATA6: now also U$37.SIGVIA1, U$37.SIGVIA3, U$38.SIGVIA1, U$38.SIGVIA3, U$39.SIGVIA1, U$39.SIGVIA3, U$40.SIGVIA1, U$40.SIGVIA3, U$41.SIGVIA1, U$41.SIGVIA3
- net DATA7: now also U$43.SIGVIA1, U$43.SIGVIA3, U$44.SIGVIA1, U$44.SIGVIA3, U$45.SIGVIA1, U$45.SIGVIA3, U$46.SIGVIA1, U$46.SIGVIA3, U$47.SIGVIA1, U$47.SIGVIA3
- net DATA8: now also U$49.SIGVIA1, U$49.SIGVIA3, U$50.SIGVIA1, U$50.SIGVIA3, U$51.SIGVIA1, U$51.SIGVIA3, U$52.SIGVIA1, U$52.SIGVIA3, U$53.SIGVIA1, U$53.SIGVIA3
- net DATA9: now also U$55.SIGVIA1, U$55.SIGVIA3, U$56.SIGVIA1, U$56.SIGVIA3, U$57.SIGVIA1, U$57.SIGVIA3, U$58.SIGVIA1, U$58.SIGVIA3, U$59.SIGVIA1, U$59.SIGVIA3
- net GND: now also U$2.GNDVIA1, U$2.GNDVIA3, U$2.GNDVIA4, U$2.GNDVIA6, U$3.GNDVIA1, U$3.GNDVIA3, U$3.GNDVIA4, U$3.GNDVIA6, U$4.GNDVIA1, U$4.GNDVIA3, U$4.GNDVIA4, U$4.GNDVIA6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
- net GND1: now also U$1.GNDVIA1, U$1.GNDVIA3, U$1.GNDVIA4, U$1.GNDVIA6, U$10.GNDVIA1, U$10.GNDVIA3, U$10.GNDVIA4, U$10.GNDVIA6, U$11.GNDVIA1, U$11.GNDVIA3, U$11.GNDVIA4, U$11.GNDVIA6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
- net GND10: now also U$61.GNDVIA1, U$61.GNDVIA3, U$61.GNDVIA4, U$61.GNDVIA6, U$62.GNDVIA1, U$62.GNDVIA3, U$62.GNDVIA4, U$62.GNDVIA6, U$63.GNDVIA1, U$63.GNDVIA3, U$63.GNDVIA4, U$63.GNDVIA6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
- net GND11: now also U$67.GNDVIA1, U$67.GNDVIA3, U$67.GNDVIA4, U$67.GNDVIA6, U$68.GNDVIA1, U$68.GNDVIA3, U$68.GNDVIA4, U$68.GNDVIA6, U$69.GNDVIA1, U$69.GNDVIA3, U$69.GNDVIA4, U$69.GNDVIA6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
- net GND12: now also U$73.GNDVIA1, U$73.GNDVIA3, U$73.GNDVIA4, U$73.GNDVIA6, U$74.GNDVIA1, U$74.GNDVIA3, U$74.GNDVIA4, U$74.GNDVIA6, U$75.GNDVIA1, U$75.GNDVIA3, U$75.GNDVIA4, U$75.GNDVIA6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
- net GND13: now also U$79.GNDVIA1, U$79.GNDVIA3, U$79.GNDVIA4, U$79.GNDVIA6, U$80.GNDVIA1, U$80.GNDVIA3, U$80.GNDVIA4, U$80.GNDVIA6, U$81.GNDVIA1, U$81.GNDVIA3, U$81.GNDVIA4, U$81.GNDVIA6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
- net GND14: now also U$85.GNDVIA1, U$85.GNDVIA3, U$85.GNDVIA4, U$85.GNDVIA6, U$86.GNDVIA1, U$86.GNDVIA3, U$86.GNDVIA4, U$86.GNDVIA6, U$87.GNDVIA1, U$87.GNDVIA3, U$87.GNDVIA4, U$87.GNDVIA6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
- net GND15: now also U$91.GNDVIA1, U$91.GNDVIA3, U$91.GNDVIA4, U$91.GNDVIA6, U$92.GNDVIA1, U$92.GNDVIA3, U$92.GNDVIA4, U$92.GNDVIA6, U$93.GNDVIA1, U$93.GNDVIA3, U$93.GNDVIA4, U$93.GNDVIA6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
- net GND4: now also U$25.GNDVIA1, U$25.GNDVIA3, U$25.GNDVIA4, U$25.GNDVIA6, U$26.GNDVIA1, U$26.GNDVIA3, U$26.GNDVIA4, U$26.GNDVIA6, U$27.GNDVIA1, U$27.GNDVIA3, U$27.GNDVIA4, U$27.GNDVIA6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
- net GND5: now also U$31.GNDVIA1, U$31.GNDVIA3, U$31.GNDVIA4, U$31.GNDVIA6, U$32.GNDVIA1, U$32.GNDVIA3, U$32.GNDVIA4, U$32.GNDVIA6, U$33.GNDVIA1, U$33.GNDVIA3, U$33.GNDVIA4, U$33.GNDVIA6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
- net GND6: now also U$37.GNDVIA1, U$37.GNDVIA3, U$37.GNDVIA4, U$37.GNDVIA6, U$38.GNDVIA1, U$38.GNDVIA3, U$38.GNDVIA4, U$38.GNDVIA6, U$39.GNDVIA1, U$39.GNDVIA3, U$39.GNDVIA4, U$39.GNDVIA6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
- net GND7: now also U$43.GNDVIA1, U$43.GNDVIA3, U$43.GNDVIA4, U$43.GNDVIA6, U$44.GNDVIA1, U$44.GNDVIA3, U$44.GNDVIA4, U$44.GNDVIA6, U$45.GNDVIA1, U$45.GNDVIA3, U$45.GNDVIA4, U$45.GNDVIA6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
- net GND8: now also U$49.GNDVIA1, U$49.GNDVIA3, U$49.GNDVIA4, U$49.GNDVIA6, U$50.GNDVIA1, U$50.GNDVIA3, U$50.GNDVIA4, U$50.GNDVIA6, U$51.GNDVIA1, U$51.GNDVIA3, U$51.GNDVIA4, U$51.GNDVIA6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
- net GND9: now also U$55.GNDVIA1, U$55.GNDVIA3, U$55.GNDVIA4, U$55.GNDVIA6, U$56.GNDVIA1, U$56.GNDVIA3, U$56.GNDVIA4, U$56.GNDVIA6, U$57.GNDVIA1, U$57.GNDVIA3, U$57.GNDVIA4, U$57.GNDVIA6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
Routing:
- net GND3: track 123.6 -> 0.00 mm, vias 18 -> 0
- net GND2: track 123.6 -> 0.00 mm, vias 18 -> 0
- net GND9: track 123.6 -> 111.7 mm, vias 18 -> 19
- net GND15: track 123.6 -> 111.7 mm, vias 18 -> 19
- net GND11: track 123.6 -> 111.7 mm, vias 18 -> 19
- net GND10: track 123.6 -> 111.7 mm, vias 18 -> 19
- net GND12: track 123.6 -> 111.7 mm, vias 18 -> 19
- net GND5: track 123.6 -> 111.7 mm, vias 18 -> 19
- net GND1: track 123.6 -> 111.7 mm, vias 18 -> 19
- net GND7: track 123.6 -> 111.7 mm, vias 18 -> 19
- net GND13: track 123.6 -> 111.7 mm, vias 18 -> 19
- net GND6: track 123.6 -> 111.7 mm, vias 18 -> 19
- net GND4: track 123.6 -> 111.7 mm, vias 18 -> 19
- net GND: track 123.6 -> 111.7 mm, vias 18 -> 19
- net GND14: track 123.6 -> 111.7 mm, vias 18 -> 19
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- removed copper zone on layer 16, net 5V2
- removed copper zone on layer 16, net 5V3
- removed copper zone on layer 1, net DATA2
- removed copper zone on layer 1, net DATA3
- removed copper zone on layer 1, net GND2
- removed copper zone on layer 1, net GND3
- removed copper zone on layer 1, net N$10
- removed copper zone on layer 1, net N$7
Other:
- board size 260 x 187.7 mm -> 260.7 x 136.2 mm
- board text added: "1"
- board text added: "10"
- board text added: "11"
- board text added: "12"
- board text added: "13"
- board text added: "14"
- board text added: "2"
- board text added: "3"
- board text added: "4"
- board text added: "5"
- board text added: "6"
- board text added: "7"
- board text added: "8"
- board text added: "9"
- board text added: "Blinkinlabs loves you!"
- board text added: "Blinkinlabs.com"
- board text added: "BlinkyTile by"
- board text added: "BlinkyTile by Blinkinlabs Revision F"
- board text added: "Designed by: Matt Mets Ethan Hartman Sam Choy Honghong Lu"
- board text added: "Enjoy!"
- board text added: "For instructions"
- board text added: "Pick me!"
- board text added: "This is a weird shape..."
- board text added: "What should go here???"
- board text added: "blinkytile.com"
- board text added: "head to:"
- board text removed: "BlinkyTile Rev. D"
- board text removed: "BlinkyTile Test Sheet - Revision D - By Blinkinlabs"
- board text removed: "Greeting from Blinkinlabs"
- board text removed: "Snap Solder Enjoy!"
- board text removed: "blinkinlabs.com"
- board text removed: "vscore"

Commit message: Rev 5 panel design by Sam
Parts:
- removed C1, C16: .1uF, adafruit:C0603
- removed E$100, E$101, E$102, E$103, E$104, E$105, E$106, E$107, E$108, E$109, E$110, E$111, E$112, E$113, E$114, E$115, E$116, E$117, E$118, E$119, E$120, E$121, E$122, E$123, E$124, E$125, E$126, E$127, E$128, E$129, E$130, E$131, E$132, E$133, E$134, E$135, E$136, E$137, E$138, E$139, E$140, E$141, E$142, E$143, E$144, E$145, E$146, E$147, E$148, E$149, E$150, E$151, E$152, E$52, E$53, E$54, E$55, E$56, E$57, E$58, E$59, E$60, E$61, E$62, E$63, E$64, E$65, E$66, E$67, E$68, E$69, E$70, E$71, E$72, E$73, E$74, E$75, E$76, E$77, E$78, E$79, E$80, E$81, E$82, E$83, E$84, E$85, E$86, E$87, E$88, E$89, E$90, E$91, E$92, E$93, E$94, E$95, E$96, E$97, E$98, E$99: (no value), dodocohedreled:MOUSE_BITE
- removed R1, R31: 75, adafruit:R0603
- removed R2, R32: 10k, adafruit:R0603
- removed U$4, U$5, U$6, U$91, U$93, U$94, U$95: D_EDGEMOD, dodocohedreled:D_EDGE_SLOT_MOD
- removed U$7, U$96: WS2822S_LED, blinkinlabs:WS2822S_LED
- added C3, C4: .1uF, adafruit:C0603
- added E$23, E$24, E$25, E$26, E$27, E$28, E$29, E$3, E$30, E$31, E$32, E$4: (no value), dodocohedreled:MOUSE_BITE_1
- added R5, R7: 75, adafruit:R0603
- added R6, R8: 10k, adafruit:R0603
- added U$13, U$14, U$15, U$16, U$17, U$19, U$20, U$21, U$22, U$23: D_EDGEMOD, dodocohedreled:D_EDGE_SLOT_MOD
- added U$18, U$24: WS2822S_LED, blinkinlabs:WS2822S_LED
- E$1, E$46, E$49: device dodocohedreled:MOUSE_BITE -> con-hdrs40:MTA-100-3V
- E$10, E$11, E$12, E$13, E$14, E$15, E$16, E$17, E$18, E$19, E$2, E$20, E$21, E$22, E$33, E$34, E$35, E$36, E$37, E$38, E$39, E$40, E$41, E$42, E$43, E$44, E$45, E$47, E$48, E$5, E$50, E$51, E$6, E$7, E$8, E$9: device dodocohedreled:MOUSE_BITE -> dodocohedreled:MOUSE_BITE_1
- moved E$2 291.3 mm to (250.8, 111.8), flipped to the bottom, turned to 0 degrees
- moved U$2 277.7 mm to (251.5, 96.5), flipped to the bottom, turned to 270 degrees
- moved U$3 267.2 mm to (266.7, 96.5), flipped to the bottom, turned to 270 degrees
- moved E$1 263.2 mm to (245.1, 96.5), flipped to the bottom, turned to 270 degrees
- moved E$16 259.3 mm to (240.0, 168.0), turned to 0 degrees
- moved U$34 232.9 mm to (252.5, 159.4), turned to 144 degrees
- moved U$58 231.3 mm to (150.9, 102.3), turned to 144 degrees
- moved E$18 223.4 mm to (255.2, 121.4), turned to 216 degrees
- moved U$32 221.7 mm to (260.2, 135.7), turned to 72 degrees
- moved E$15 219.5 mm to (204.4, 121.4), turned to 216 degrees
- moved U$56 213.3 mm to (158.6, 78.6), turned to 72 degrees
- moved E$7 211.6 mm to (87.6, 168.0), turned to 0 degrees
- moved E$13 204.8 mm to (189.2, 168.0)
- moved E$46 204.1 mm to (260.4, 96.5), flipped to the bottom, turned to 270 degrees
- moved R12 201.4 mm to (241.6, 147.6), turned to 90 degrees
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Connections:
- net 5V1 renamed 5V2
- removed net 5V: R1.1, U$2.P$2, U$2.P$4, U$2.P$7, U$2.P$9, U$2.PWRVIA1, U$2.PWRVIA3, U$2.PWRVIA4, U$2.PWRVIA6, U$3.P$2, U$3.P$4, U$3.P$7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
- removed net ADRI: U$7.2
- removed net ADRI15: U$96.2
- removed net DATA: R2.2, U$2.P$3, U$2.P$8, U$2.SIGVIA1, U$2.SIGVIA3, U$3.P$3, U$3.P$8, U$3.SIGVIA1, U$3.SIGVIA3, U$4.P$3, U$4.P$8, U$4.SIGVIA1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
- removed net DATA15: R32.2, U$91.P$3, U$91.P$8, U$91.SIGVIA1, U$91.SIGVIA3, U$92.P$3, U$92.P$8, U$92.SIGVIA1, U$92.SIGVIA3, U$93.P$3, U$93.P$8, U$93.SIGVIA1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
- removed net GND: C1.2, U$2.GNDVIA1, U$2.GNDVIA3, U$2.GNDVIA4, U$2.GNDVIA6, U$2.P$1, U$2.P$10, U$2.P$5, U$2.P$6, U$3.GNDVIA1, U$3.GNDVIA3, U$3.GNDVIA4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
- removed net GND15: C16.2, U$91.GNDVIA1, U$91.GNDVIA3, U$91.GNDVIA4, U$91.GNDVIA6, U$91.P$1, U$91.P$10, U$91.P$5, U$91.P$6, U$92.GNDVIA1, U$92.GNDVIA3, U$92.GNDVIA4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
- removed net N$1: C1.1, R1.2, U$7.3
- removed net N$2: R2.1, U$7.1
- removed net N$47: C16.1, R31.2, U$96.3
- removed net N$48: R32.1, U$96.1
- new net 5V3: R5.1, U$13.P$2, U$13.P$4, U$13.P$7, U$13.P$9, U$13.PWRVIA1, U$13.PWRVIA3, U$13.PWRVIA4, U$13.PWRVIA6, U$14.P$2, U$14.P$4, U$14.P$7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
- new net ADRI2: U$18.2
- new net ADRI3: U$24.2
- new net DATA2: R6.2, U$13.P$3, U$13.P$8, U$13.SIGVIA1, U$13.SIGVIA3, U$14.P$3, U$14.P$8, U$14.SIGVIA1, U$14.SIGVIA3, U$15.P$3, U$15.P$8, U$15.SIGVIA1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
- new net DATA3: R8.2, U$19.P$3, U$19.P$8, U$19.SIGVIA1, U$19.SIGVIA3, U$20.P$3, U$20.P$8, U$20.SIGVIA1, U$20.SIGVIA3, U$21.P$3, U$21.P$8, U$21.SIGVIA1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
- new net GND2: C3.2, U$13.GNDVIA1, U$13.GNDVIA3, U$13.GNDVIA4, U$13.GNDVIA6, U$13.P$1, U$13.P$10, U$13.P$5, U$13.P$6, U$14.GNDVIA1, U$14.GNDVIA3, U$14.GNDVIA4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
- new net GND3: C4.2, U$19.GNDVIA1, U$19.GNDVIA3, U$19.GNDVIA4, U$19.GNDVIA6, U$19.P$1, U$19.P$10, U$19.P$5, U$19.P$6, U$20.GNDVIA1, U$20.GNDVIA3, U$20.GNDVIA4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
- new net N$11: C4.1, R7.2, U$24.3
- new net N$12: R8.1, U$24.1
- new net N$8: C3.1, R5.2, U$18.3
- new net N$9: R6.1, U$18.1
- new net S$1: E$1.2, U$2.P$3
- new net S$2: E$1.3, U$2.P$1, U$2.P$5
- new net S$3: E$1.1, U$2.P$7, U$2.P$9
- new net S$4: E$49.2, U$92.P$3
- new net S$5: E$49.3, U$92.P$1, U$92.P$5
- new net S$6: E$49.1, U$92.P$7, U$92.P$9
- new net S$7: E$46.2, U$3.P$3
- new net S$8: E$46.3, U$3.P$1, U$3.P$5
- new net S$9: E$46.1, U$3.P$7, U$3.P$9
- net 5V10: now also R19.1, U$55.P$2, U$55.P$4, U$55.P$7, U$55.P$9, U$55.PWRVIA1, U$55.PWRVIA3, U$55.PWRVIA4, U$55.PWRVIA6, U$56.P$2, U$56.P$4, U$56.P$7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; no longer R21.1, U$61.P$2, U$61.P$4, U$61.P$7, U$61.P$9, U$61.PWRVIA1, U$61.PWRVIA3, U$61.PWRVIA4, U$61.PWRVIA6, U$62.P$2, U$62.P$4, U$62.P$7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
- net 5V11: now also R21.1, U$61.P$2, U$61.P$4, U$61.P$7, U$61.P$9, U$61.PWRVIA1, U$61.PWRVIA3, U$61.PWRVIA4, U$61.PWRVIA6, U$62.P$2, U$62.P$4, U$62.P$7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; no longer R23.1, U$67.P$2, U$67.P$4, U$67.P$7, U$67.P$9, U$67.PWRVIA1, U$67.PWRVIA3, U$67.PWRVIA4, U$67.PWRVIA6, U$68.P$2, U$68.P$4, U$68.P$7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
- net 5V12: now also R23.1, U$67.P$2, U$67.P$4, U$67.P$7, U$67.P$9, U$67.PWRVIA1, U$67.PWRVIA3, U$67.PWRVIA4, U$67.PWRVIA6, U$68.P$2, U$68.P$4, U$68.P$7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; no longer R25.1, U$73.P$2, U$73.P$4, U$73.P$7, U$73.P$9, U$73.PWRVIA1, U$73.PWRVIA3, U$73.PWRVIA4, U$73.PWRVIA6, U$74.P$2, U$74.P$4, U$74.P$7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
- net 5V13: now also R25.1, U$73.P$2, U$73.P$4, U$73.P$7, U$73.P$9, U$73.PWRVIA1, U$73.PWRVIA3, U$73.PWRVIA4, U$73.PWRVIA6, U$74.P$2, U$74.P$4, U$74.P$7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; no longer R27.1, U$79.P$2, U$79.P$4, U$79.P$7, U$79.P$9, U$79.PWRVIA1, U$79.PWRVIA3, U$79.PWRVIA4, U$79.PWRVIA6, U$80.P$2, U$80.P$4, U$80.P$7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
- net 5V14: now also R27.1, U$79.P$2, U$79.P$4, U$79.P$7, U$79.P$9, U$79.PWRVIA1, U$79.PWRVIA3, U$79.PWRVIA4, U$79.PWRVIA6, U$80.P$2, U$80.P$4, U$80.P$7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; no longer R29.1, U$85.P$2, U$85.P$4, U$85.P$7, U$85.P$9, U$85.PWRVIA1, U$85.PWRVIA3, U$85.PWRVIA4, U$85.PWRVIA6, U$86.P$2, U$86.P$4, U$86.P$7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
- net 5V15: now also R29.1, U$85.P$2, U$85.P$4, U$85.P$7, U$85.P$9, U$85.PWRVIA1, U$85.PWRVIA3, U$85.PWRVIA4, U$85.PWRVIA6, U$86.P$2, U$86.P$4, U$86.P$7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; no longer R31.1, U$91.P$2, U$91.P$4, U$91.P$7, U$91.P$9, U$91.PWRVIA1, U$91.PWRVIA3, U$91.PWRVIA4, U$91.PWRVIA6, U$92.P$2, U$92.P$4, U$92.P$7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
- net 5V4: now also R7.1, U$19.P$2, U$19.P$4, U$19.P$7, U$19.P$9, U$19.PWRVIA1, U$19.PWRVIA3, U$19.PWRVIA4, U$19.PWRVIA6, U$20.P$2, U$20.P$4, U$20.P$7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; no longer R9.1, U$25.P$2, U$25.P$4, U$25.P$7, U$25.P$9, U$25.PWRVIA1, U$25.PWRVIA3, U$25.PWRVIA4, U$25.PWRVIA6, U$26.P$2, U$26.P$4, U$26.P$7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
- net 5V5: now also R9.1, U$25.P$2, U$25.P$4, U$25.P$7, U$25.P$9, U$25.PWRVIA1, U$25.PWRVIA3, U$25.PWRVIA4, U$25.PWRVIA6, U$26.P$2, U$26.P$4, U$26.P$7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; no longer R11.1, U$31.P$2, U$31.P$4, U$31.P$7, U$31.P$9, U$31.PWRVIA1, U$31.PWRVIA3, U$31.PWRVIA4, U$31.PWRVIA6, U$32.P$2, U$32.P$4, U$32.P$7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
- net 5V6: now also R11.1, U$31.P$2, U$31.P$4, U$31.P$7, U$31.P$9, U$31.PWRVIA1, U$31.PWRVIA3, U$31.PWRVIA4, U$31.PWRVIA6, U$32.P$2, U$32.P$4, U$32.P$7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; no longer R13.1, U$37.P$2, U$37.P$4, U$37.P$7, U$37.P$9, U$37.PWRVIA1, U$37.PWRVIA3, U$37.PWRVIA4, U$37.PWRVIA6, U$38.P$2, U$38.P$4, U$38.P$7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
- net 5V7: now also R13.1, U$37.P$2, U$37.P$4, U$37.P$7, U$37.P$9, U$37.PWRVIA1, U$37.PWRVIA3, U$37.PWRVIA4, U$37.PWRVIA6, U$38.P$2, U$38.P$4, U$38.P$7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; no longer R15.1, U$43.P$2, U$43.P$4, U$43.P$7, U$43.P$9, U$43.PWRVIA1, U$43.PWRVIA3, U$43.PWRVIA4, U$43.PWRVIA6, U$44.P$2, U$44.P$4, U$44.P$7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
- net 5V8: now also R15.1, U$43.P$2, U$43.P$4, U$43.P$7, U$43.P$9, U$43.PWRVIA1, U$43.PWRVIA3, U$43.PWRVIA4, U$43.PWRVIA6, U$44.P$2, U$44.P$4, U$44.P$7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; no longer R17.1, U$49.P$2, U$49.P$4, U$49.P$7, U$49.P$9, U$49.PWRVIA1, U$49.PWRVIA3, U$49.PWRVIA4, U$49.PWRVIA6, U$50.P$2, U$50.P$4, U$50.P$7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
- net 5V9: now also R17.1, U$49.P$2, U$49.P$4, U$49.P$7, U$49.P$9, U$49.PWRVIA1, U$49.PWRVIA3, U$49.PWRVIA4, U$49.PWRVIA6, U$50.P$2, U$50.P$4, U$50.P$7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; no longer R19.1, U$55.P$2, U$55.P$4, U$55.P$7, U$55.P$9, U$55.PWRVIA1, U$55.PWRVIA3, U$55.PWRVIA4, U$55.PWRVIA6, U$56.P$2, U$56.P$4, U$56.P$7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
Routing:
- net GND2: track 0.00 -> 111.7 mm, vias 0 -> 19
- net GND3: track 0.00 -> 111.7 mm, vias 0 -> 19
- net GND15: track 111.7 -> 0.00 mm, vias 19 -> 0
- net GND: track 111.7 -> 0.00 mm, vias 19 -> 0
- net DATA3: track 0.00 -> 15.3 mm
- net DATA15: track 15.3 -> 0.00 mm
- net DATA2: track 0.00 -> 15.3 mm
- net DATA: track 15.3 -> 0.00 mm
- net ADRI15: track 5.78 -> 0.00 mm, vias 1 -> 0
- net ADRI: track 5.78 -> 0.00 mm, vias 1 -> 0
- net ADRI3: track 0.00 -> 5.78 mm, vias 0 -> 1
- net ADRI2: track 0.00 -> 5.78 mm, vias 0 -> 1
- net S$7: track 0.00 -> 5.62 mm
- net S$4: track 0.00 -> 5.62 mm
- net S$1: track 0.00 -> 5.62 mm
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- added copper zone on layer 16, net 5V3
- added copper zone on layer 1, net DATA2
- added copper zone on layer 1, net DATA3
- added copper zone on layer 1, net GND2
- added copper zone on layer 1, net GND3
- added copper zone on layer 1, net N$10
- added copper zone on layer 1, net N$7
- added copper zone on layer 16, net S$2
- added copper zone on layer 1, net S$3
- added copper zone on layer 16, net S$5
- added copper zone on layer 1, net S$6
- added copper zone on layer 16, net S$8
- added copper zone on layer 1, net S$9
- removed copper zone on layer 16, net 5V
- removed copper zone on layer 1, net DATA
- removed copper zone on layer 1, net DATA15
- removed copper zone on layer 1, net GND
- removed copper zone on layer 1, net GND15
- removed copper zone on layer 1, net N$4
- removed copper zone on layer 1, net N$46
Other:
- board size 260.7 x 136.2 mm -> 276.9 x 177.8 mm
- board text added: "+5V"
- board text added: "01"
- board text added: "02"
- board text added: "03"
- board text added: "04"
- board text added: "05"
- board text added: "06"
- board text added: "07"
- board text added: "08"
- board text added: "09"
- board text added: "BlinkyTile Revision H"
- board text added: "Designed by: Matt Mets, Ethan Hartman, Sam Choy, Honghong Lu"
- board text added: "GND"
- board text added: "SIG"
- board text removed: "1"
- board text removed: "2"
- board text removed: "3"
- board text removed: "4"
- board text removed: "5"
- board text removed: "6"
- board text removed: "7"
- board text removed: "8"
- board text removed: "9"
- board text removed: "Blinkinlabs loves you!"
- board text removed: "BlinkyTile by Blinkinlabs Revision F"
- board text removed: "Designed by: Matt Mets Ethan Hartman Sam Choy Honghong Lu"
- board text removed: "Enjoy!"
- board text removed: "For instructions"
- board text removed: "Pick me!"
- board text removed: "This is a weird shape..."
- board text removed: "What should go here???"
- board text removed: "blinkytile.com"
- board text removed: "head to:"

Commit message: Rev 6 panel design (as submitted for prototype PCB)
Parts:
- removed C15: .1uF, adafruit:C0603
- removed R29: 75, adafruit:R0603
- removed R30: 10k, adafruit:R0603
- removed U$87, U$88, U$89, U$92: D_EDGEMOD, dodocohedreled:D_EDGE_SLOT_MOD
- removed U$90: WS2822S_LED, blinkinlabs:WS2822S_LED
- added C1: .1uF, adafruit:C0603
- added E$52: (no value), con-hdrs40:MTA-100-3V
- added E$53, E$54, E$55, E$56, E$57, E$58, E$59, E$60, E$61, E$62, E$63, E$64, E$65, E$66, E$67, E$68, E$69, E$70, E$71, E$72, E$73, E$74, E$75, E$76, E$77, E$78, E$79, E$80, E$81, E$82, E$83, E$84, E$85, E$86, E$87, E$88, E$89, E$90: (no value), dodocohedreled:MOUSE_BITE_1
- added R1: 75, adafruit:R0603
- added R2: 10k, adafruit:R0603
- added U$4, U$5, U$6: D_EDGEMOD, dodocohedreled:D_EDGE_SLOT_MOD
- added U$7: WS2822S_LED, blinkinlabs:WS2822S_LED
- E$1, E$46: device con-hdrs40:MTA-100-3V -> dodocohedreled:MOUSE_BITE_1
- U$54, U$60, U$66, U$72, U$78, U$84: value WS2822S_LED -> D_EDGEMOD; device blinkinlabs:WS2822S_LED -> dodocohedreled:D_EDGE_SLOT_MOD
- U$56, U$62, U$68, U$74, U$80, U$86: value D_EDGEMOD -> WS2822S_LED; device dodocohedreled:D_EDGE_SLOT_MOD -> blinkinlabs:WS2822S_LED
- moved E$2 390.7 mm to (-91.4, -76.8), flipped to the top, turned to 144 degrees
- moved E$48 388.9 mm to (-100.8, -47.8), flipped to the top, turned to 72 degrees
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Connections:
- removed net 5V15: R29.1, U$85.P$2, U$85.P$4, U$85.P$7, U$85.P$9, U$85.PWRVIA1, U$85.PWRVIA3, U$85.PWRVIA4, U$85.PWRVIA6, U$86.P$2, U$86.P$4, U$86.P$7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
- removed net N$44: C15.1, R29.2, U$90.3
- removed net N$45: R30.1, U$90.1
- removed net S$1: E$1.2, U$2.P$3
- removed net S$2: E$1.3, U$2.P$1, U$2.P$5
- removed net S$3: E$1.1, U$2.P$7, U$2.P$9
- new net 5V1: R3.1, U$1.P$2, U$1.P$4, U$1.P$7, U$1.P$9, U$1.PWRVIA1, U$1.PWRVIA3, U$1.PWRVIA4, U$1.PWRVIA6, U$10.P$2, U$10.P$4, U$10.P$7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
- new net N$2: C1.1, R1.2, U$7.3
- new net N$4: R2.1, U$7.1
- net 5V10: now also U$60.P$2, U$60.P$4, U$60.P$7, U$60.P$9, U$60.PWRVIA1, U$60.PWRVIA3, U$60.PWRVIA4, U$60.PWRVIA6, U$61.P$2, U$61.P$4, U$61.P$7, U$61.P$9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; no longer U$55.P$2, U$55.P$4, U$55.P$7, U$55.P$9, U$55.PWRVIA1, U$55.PWRVIA3, U$55.PWRVIA4, U$55.PWRVIA6, U$56.P$2, U$56.P$4, U$56.P$7, U$56.P$9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
- net 5V11: now also U$66.P$2, U$66.P$4, U$66.P$7, U$66.P$9, U$66.PWRVIA1, U$66.PWRVIA3, U$66.PWRVIA4, U$66.PWRVIA6, U$67.P$2, U$67.P$4, U$67.P$7, U$67.P$9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; no longer U$61.P$2, U$61.P$4, U$61.P$7, U$61.P$9, U$61.PWRVIA1, U$61.PWRVIA3, U$61.PWRVIA4, U$61.PWRVIA6, U$62.P$2, U$62.P$4, U$62.P$7, U$62.P$9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
- net 5V12: now also U$72.P$2, U$72.P$4, U$72.P$7, U$72.P$9, U$72.PWRVIA1, U$72.PWRVIA3, U$72.PWRVIA4, U$72.PWRVIA6, U$73.P$2, U$73.P$4, U$73.P$7, U$73.P$9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; no longer U$67.P$2, U$67.P$4, U$67.P$7, U$67.P$9, U$67.PWRVIA1, U$67.PWRVIA3, U$67.PWRVIA4, U$67.PWRVIA6, U$68.P$2, U$68.P$4, U$68.P$7, U$68.P$9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
- net 5V13: now also U$78.P$2, U$78.P$4, U$78.P$7, U$78.P$9, U$78.PWRVIA1, U$78.PWRVIA3, U$78.PWRVIA4, U$78.PWRVIA6, U$79.P$2, U$79.P$4, U$79.P$7, U$79.P$9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; no longer U$73.P$2, U$73.P$4, U$73.P$7, U$73.P$9, U$73.PWRVIA1, U$73.PWRVIA3, U$73.PWRVIA4, U$73.PWRVIA6, U$74.P$2, U$74.P$4, U$74.P$7, U$74.P$9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
- net 5V14: now also U$84.P$2, U$84.P$4, U$84.P$7, U$84.P$9, U$84.PWRVIA1, U$84.PWRVIA3, U$84.PWRVIA4, U$84.PWRVIA6, U$85.P$2, U$85.P$4, U$85.P$7, U$85.P$9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; no longer U$79.P$2, U$79.P$4, U$79.P$7, U$79.P$9, U$79.PWRVIA1, U$79.PWRVIA3, U$79.PWRVIA4, U$79.PWRVIA6, U$80.P$2, U$80.P$4, U$80.P$7, U$80.P$9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
- net 5V2: now also R5.1, U$13.P$2, U$13.P$4, U$13.P$7, U$13.P$9, U$13.PWRVIA1, U$13.PWRVIA3, U$13.PWRVIA4, U$13.PWRVIA6, U$14.P$2, U$14.P$4, U$14.P$7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; no longer R3.1, U$1.P$2, U$1.P$4, U$1.P$7, U$1.P$9, U$1.PWRVIA1, U$1.PWRVIA3, U$1.PWRVIA4, U$1.PWRVIA6, U$10.P$2, U$10.P$4, U$10.P$7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
- net 5V3: now also R7.1, U$19.P$2, U$19.P$4, U$19.P$7, U$19.P$9, U$19.PWRVIA1, U$19.PWRVIA3, U$19.PWRVIA4, U$19.PWRVIA6, U$20.P$2, U$20.P$4, U$20.P$7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; no longer R5.1, U$13.P$2, U$13.P$4, U$13.P$7, U$13.P$9, U$13.PWRVIA1, U$13.PWRVIA3, U$13.PWRVIA4, U$13.PWRVIA6, U$14.P$2, U$14.P$4, U$14.P$7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
- net 5V4: now also R9.1, U$25.P$2, U$25.P$4, U$25.P$7, U$25.P$9, U$25.PWRVIA1, U$25.PWRVIA3, U$25.PWRVIA4, U$25.PWRVIA6, U$26.P$2, U$26.P$4, U$26.P$7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; no longer R7.1, U$19.P$2, U$19.P$4, U$19.P$7, U$19.P$9, U$19.PWRVIA1, U$19.PWRVIA3, U$19.PWRVIA4, U$19.PWRVIA6, U$20.P$2, U$20.P$4, U$20.P$7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
- net 5V5: now also R11.1, U$31.P$2, U$31.P$4, U$31.P$7, U$31.P$9, U$31.PWRVIA1, U$31.PWRVIA3, U$31.PWRVIA4, U$31.PWRVIA6, U$32.P$2, U$32.P$4, U$32.P$7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; no longer R9.1, U$25.P$2, U$25.P$4, U$25.P$7, U$25.P$9, U$25.PWRVIA1, U$25.PWRVIA3, U$25.PWRVIA4, U$25.PWRVIA6, U$26.P$2, U$26.P$4, U$26.P$7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
- net 5V6: now also R13.1, U$37.P$2, U$37.P$4, U$37.P$7, U$37.P$9, U$37.PWRVIA1, U$37.PWRVIA3, U$37.PWRVIA4, U$37.PWRVIA6, U$38.P$2, U$38.P$4, U$38.P$7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; no longer R11.1, U$31.P$2, U$31.P$4, U$31.P$7, U$31.P$9, U$31.PWRVIA1, U$31.PWRVIA3, U$31.PWRVIA4, U$31.PWRVIA6, U$32.P$2, U$32.P$4, U$32.P$7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
- net 5V7: now also R15.1, U$43.P$2, U$43.P$4, U$43.P$7, U$43.P$9, U$43.PWRVIA1, U$43.PWRVIA3, U$43.PWRVIA4, U$43.PWRVIA6, U$44.P$2, U$44.P$4, U$44.P$7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; no longer R13.1, U$37.P$2, U$37.P$4, U$37.P$7, U$37.P$9, U$37.PWRVIA1, U$37.PWRVIA3, U$37.PWRVIA4, U$37.PWRVIA6, U$38.P$2, U$38.P$4, U$38.P$7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
- net 5V8: now also R1.1, U$2.P$2, U$2.P$4, U$2.P$7, U$2.P$9, U$2.PWRVIA1, U$2.PWRVIA3, U$2.PWRVIA4, U$2.PWRVIA6, U$3.P$2, U$3.P$4, U$3.P$7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; no longer R15.1, U$43.P$2, U$43.P$4, U$43.P$7, U$43.P$9, U$43.PWRVIA1, U$43.PWRVIA3, U$43.PWRVIA4, U$43.PWRVIA6, U$44.P$2, U$44.P$4, U$44.P$7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
- net 5V9: now also U$54.P$2, U$54.P$4, U$54.P$7, U$54.P$9, U$54.PWRVIA1, U$54.PWRVIA3, U$54.PWRVIA4, U$54.PWRVIA6, U$55.P$2, U$55.P$4, U$55.P$7, U$55.P$9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; no longer U$49.P$2, U$49.P$4, U$49.P$7, U$49.P$9, U$49.PWRVIA1, U$49.PWRVIA3, U$49.PWRVIA4, U$49.PWRVIA6, U$50.P$2, U$50.P$4, U$50.P$7, U$50.P$9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
- net ADRI10: now also U$62.2; no longer U$66.2
- net ADRI11: now also U$68.2; no longer U$72.2
- net ADRI12: now also U$74.2; no longer U$78.2
- net ADRI13: now also U$80.2; no longer U$84.2
- net ADRI14: now also U$86.2; no longer U$90.2
- net ADRI8: now also U$7.2; no longer U$54.2
- net ADRI9: now also U$56.2; no longer U$60.2
- net DATA10: now also R20.2, U$57.P$3, U$57.P$8, U$57.SIGVIA1, U$57.SIGVIA3, U$58.P$3, U$58.P$8, U$58.SIGVIA1, U$58.SIGVIA3, U$59.P$3, U$59.P$8, U$59.SIGVIA1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; no longer R22.2, U$62.P$3, U$62.P$8, U$62.SIGVIA1, U$62.SIGVIA3, U$63.P$3, U$63.P$8, U$63.SIGVIA1, U$63.SIGVIA3, U$64.P$3, U$64.P$8, U$64.SIGVIA1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
- net DATA11: now also R22.2, U$63.P$3, U$63.P$8, U$63.SIGVIA1, U$63.SIGVIA3, U$64.P$3, U$64.P$8, U$64.SIGVIA1, U$64.SIGVIA3, U$65.P$3, U$65.P$8, U$65.SIGVIA1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; no longer R24.2, U$68.P$3, U$68.P$8, U$68.SIGVIA1, U$68.SIGVIA3, U$69.P$3, U$69.P$8, U$69.SIGVIA1, U$69.SIGVIA3, U$70.P$3, U$70.P$8, U$70.SIGVIA1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
- net DATA12: now also R24.2, U$69.P$3, U$69.P$8, U$69.SIGVIA1, U$69.SIGVIA3, U$70.P$3, U$70.P$8, U$70.SIGVIA1, U$70.SIGVIA3, U$71.P$3, U$71.P$8, U$71.SIGVIA1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; no longer R26.2, U$74.P$3, U$74.P$8, U$74.SIGVIA1, U$74.SIGVIA3, U$75.P$3, U$75.P$8, U$75.SIGVIA1, U$75.SIGVIA3, U$76.P$3, U$76.P$8, U$76.SIGVIA1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
- net DATA13: now also R26.2, U$75.P$3, U$75.P$8, U$75.SIGVIA1, U$75.SIGVIA3, U$76.P$3, U$76.P$8, U$76.SIGVIA1, U$76.SIGVIA3, U$77.P$3, U$77.P$8, U$77.SIGVIA1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; no longer R28.2, U$80.P$3, U$80.P$8, U$80.SIGVIA1, U$80.SIGVIA3, U$81.P$3, U$81.P$8, U$81.SIGVIA1, U$81.SIGVIA3, U$82.P$3, U$82.P$8, U$82.SIGVIA1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
- net DATA14: now also R28.2, U$81.P$3, U$81.P$8, U$81.SIGVIA1, U$81.SIGVIA3, U$82.P$3, U$82.P$8, U$82.SIGVIA1, U$82.SIGVIA3, U$83.P$3, U$83.P$8, U$83.SIGVIA1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; no longer R30.2, U$86.P$3, U$86.P$8, U$86.SIGVIA1, U$86.SIGVIA3, U$87.P$3, U$87.P$8, U$87.SIGVIA1, U$87.SIGVIA3, U$88.P$3, U$88.P$8, U$88.SIGVIA1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
- net DATA8: now also R2.2, U$2.P$3, U$2.P$8, U$2.SIGVIA1, U$2.SIGVIA3, U$3.P$3, U$3.P$8, U$3.SIGVIA1, U$3.SIGVIA3, U$4.P$3, U$4.P$8, U$4.SIGVIA1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; no longer R18.2, U$49.P$3, U$49.P$8, U$49.SIGVIA1, U$49.SIGVIA3, U$50.P$3, U$50.P$8, U$50.SIGVIA1, U$50.SIGVIA3, U$51.P$3, U$51.P$8, U$51.SIGVIA1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
- net DATA9: now also R18.2, U$51.P$3, U$51.P$8, U$51.SIGVIA1, U$51.SIGVIA3, U$52.P$3, U$52.P$8, U$52.SIGVIA1, U$52.SIGVIA3, U$53.P$3, U$53.P$8, U$53.SIGVIA1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; no longer R20.2, U$56.P$3, U$56.P$8, U$56.SIGVIA1, U$56.SIGVIA3, U$57.P$3, U$57.P$8, U$57.SIGVIA1, U$57.SIGVIA3, U$58.P$3, U$58.P$8, U$58.SIGVIA1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
- net GND10: now also C10.2, U$57.GNDVIA1, U$57.GNDVIA3, U$57.GNDVIA4, U$57.GNDVIA6, U$57.P$1, U$57.P$10, U$57.P$5, U$57.P$6, U$58.GNDVIA1, U$58.GNDVIA3, U$58.GNDVIA4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; no longer C11.2, U$62.GNDVIA1, U$62.GNDVIA3, U$62.GNDVIA4, U$62.GNDVIA6, U$62.P$1, U$62.P$10, U$62.P$5, U$62.P$6, U$63.GNDVIA1, U$63.GNDVIA3, U$63.GNDVIA4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
- net GND11: now also C11.2, U$63.GNDVIA1, U$63.GNDVIA3, U$63.GNDVIA4, U$63.GNDVIA6, U$63.P$1, U$63.P$10, U$63.P$5, U$63.P$6, U$64.GNDVIA1, U$64.GNDVIA3, U$64.GNDVIA4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; no longer C12.2, U$68.GNDVIA1, U$68.GNDVIA3, U$68.GNDVIA4, U$68.GNDVIA6, U$68.P$1, U$68.P$10, U$68.P$5, U$68.P$6, U$69.GNDVIA1, U$69.GNDVIA3, U$69.GNDVIA4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
- net GND12: now also C12.2, U$69.GNDVIA1, U$69.GNDVIA3, U$69.GNDVIA4, U$69.GNDVIA6, U$69.P$1, U$69.P$10, U$69.P$5, U$69.P$6, U$70.GNDVIA1, U$70.GNDVIA3, U$70.GNDVIA4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; no longer C13.2, U$74.GNDVIA1, U$74.GNDVIA3, U$74.GNDVIA4, U$74.GNDVIA6, U$74.P$1, U$74.P$10, U$74.P$5, U$74.P$6, U$75.GNDVIA1, U$75.GNDVIA3, U$75.GNDVIA4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
- net GND13: now also C13.2, U$75.GNDVIA1, U$75.GNDVIA3, U$75.GNDVIA4, U$75.GNDVIA6, U$75.P$1, U$75.P$10, U$75.P$5, U$75.P$6, U$76.GNDVIA1, U$76.GNDVIA3, U$76.GNDVIA4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; no longer C14.2, U$80.GNDVIA1, U$80.GNDVIA3, U$80.GNDVIA4, U$80.GNDVIA6, U$80.P$1, U$80.P$10, U$80.P$5, U$80.P$6, U$81.GNDVIA1, U$81.GNDVIA3, U$81.GNDVIA4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
- net GND14: now also C14.2, U$81.GNDVIA1, U$81.GNDVIA3, U$81.GNDVIA4, U$81.GNDVIA6, U$81.P$1, U$81.P$10, U$81.P$5, U$81.P$6, U$82.GNDVIA1, U$82.GNDVIA3, U$82.GNDVIA4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; no longer C15.2, U$86.GNDVIA1, U$86.GNDVIA3, U$86.GNDVIA4, U$86.GNDVIA6, U$86.P$1, U$86.P$10, U$86.P$5, U$86.P$6, U$87.GNDVIA1, U$87.GNDVIA3, U$87.GNDVIA4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
- net GND8: now also C1.2, U$2.GNDVIA1, U$2.GNDVIA3, U$2.GNDVIA4, U$2.GNDVIA6, U$2.P$1, U$2.P$10, U$2.P$5, U$2.P$6, U$3.GNDVIA1, U$3.GNDVIA3, U$3.GNDVIA4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; no longer C9.2, U$49.GNDVIA1, U$49.GNDVIA3, U$49.GNDVIA4, U$49.GNDVIA6, U$49.P$1, U$49.P$10, U$49.P$5, U$49.P$6, U$50.GNDVIA1, U$50.GNDVIA3, U$50.GNDVIA4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
- net GND9: now also C9.2, U$51.GNDVIA1, U$51.GNDVIA3, U$51.GNDVIA4, U$51.GNDVIA6, U$51.P$1, U$51.P$10, U$51.P$5, U$51.P$6, U$52.GNDVIA1, U$52.GNDVIA3, U$52.GNDVIA4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; no longer C10.2, U$56.GNDVIA1, U$56.GNDVIA3, U$56.GNDVIA4, U$56.GNDVIA6, U$56.P$1, U$56.P$10, U$56.P$5, U$56.P$6, U$57.GNDVIA1, U$57.GNDVIA3, U$57.GNDVIA4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
- net N$26: now also U$56.3; no longer U$54.3
- net N$27: now also U$56.1; no longer U$54.1
- net N$29: now also U$62.3; no longer U$60.3
- net N$30: now also U$62.1; no longer U$60.1
- net N$32: now also U$68.3; no longer U$66.3
- net N$33: now also U$68.1; no longer U$66.1
- net N$35: now also U$74.3; no longer U$72.3
- net N$36: now also U$74.1; no longer U$72.1
- net N$38: now also U$80.3; no longer U$78.3
- net N$39: now also U$80.1; no longer U$78.1
- net N$41: now also U$86.3; no longer U$84.3
- net N$42: now also U$86.1; no longer U$84.1
- net S$4: now also U$49.P$3; no longer U$92.P$3
- net S$5: now also U$49.P$1, U$49.P$5; no longer U$92.P$1, U$92.P$5
- net S$6: now also U$49.P$7, U$49.P$9; no longer U$92.P$7, U$92.P$9
- net S$7: now also E$52.2, U$50.P$3; no longer E$46.2, U$3.P$3
- net S$8: now also E$52.3, U$50.P$1, U$50.P$5; no longer E$46.3, U$3.P$1, U$3.P$5
- net S$9: now also E$52.1, U$50.P$7, U$50.P$9; no longer E$46.1, U$3.P$7, U$3.P$9
Routing:
- net S$1: track 5.62 -> 0.00 mm
- net N$44: track 3.70 -> 0.00 mm
- net N$2: track 0.00 -> 3.70 mm
- net 5V15: track 3.08 -> 0.00 mm, vias 2 -> 0
- net 5V1: track 0.00 -> 3.08 mm, vias 0 -> 2
- net N$45: track 2.10 -> 0.00 mm
- net N$4: track 0.00 -> 2.10 mm
- added copper zone on layer 16, net 5V1
- added copper zone on layer 1, net N$1
- added copper zone on layer 1, net S$5
- added copper zone on layer 16, net S$6
- added copper zone on layer 1, net S$8
- added copper zone on layer 16, net S$9
- removed copper zone on layer 16, net 5V15
- removed copper zone on layer 1, net N$43
- removed copper zone on layer 16, net S$2
- removed copper zone on layer 1, net S$3
- removed copper zone on layer 16, net S$5
- removed copper zone on layer 1, net S$6
- removed copper zone on layer 16, net S$8
- removed copper zone on layer 1, net S$9
Other:
- board size 276.9 x 177.8 mm -> 208.3 x 182.9 mm
- board text added: "1"
- board text added: "2"
- board text added: "3"
- board text added: "4"
- board text added: "5"
- board text added: "6"
- board text added: "7"
- board text added: "8"
- board text added: "9"
- board text added: "BlinkyTile Revision I"
- board text added: "For instructions head to: blinkytile.com"
- board text added: "blinkytile.com"
- board text removed: "01"
- board text removed: "02"
- board text removed: "03"
- board text removed: "04"
- board text removed: "05"
- board text removed: "06"
- board text removed: "07"
- board text removed: "08"
- board text removed: "09"
- board text removed: "BlinkyTile Revision H"
