File: controller_testjig/pcb/controller testjig.brd (EAGLE design)
At the start: 70 x 100 mm, 46 parts, among them IC1 AD8041R, J1 POWER_JACKPTH, SW2 BUTTON_2

Commit message: Update production test to minimal working function
Connections:
- net TARGET_USB_D+: now also U$1.5, U$3.D+; no longer U$1.6, U$3.D-
- net TARGET_USB_D-: now also U$1.6, U$3.D-; no longer U$1.5, U$3.D+
Routing:
- net TARGET_USB_D-: track 55.8 -> 48.8 mm
- net TARGET_USB_D+: track 48.8 -> 55.8 mm
- net N$1: track 3.52 -> 5.52 mm
Changed lines of the file:
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@@
 <via x="54.53" y="56" extent="1-16" drill="0.6" shape="square"/>
 </signal>
-<signal name="TARGET_USB_D-">
+<signal name="TARGET_USB_D+">
 <contactref element="U$1" pad="5"/>
 <contactref element="U$3" pad="D+"/>
@@
 <wire x1="17" y1="53" x2="18" y2="53" width="0.254" layer="16"/>
 </signal>
-<signal name="TARGET_USB_D+">
+<signal name="TARGET_USB_D-">
 <contactref element="U$1" pad="6"/>
 <contactref element="U$3" pad="D-"/>
@@
 <wire x1="11.135" y1="81.715" x2="10.85" y2="82" width="0.254" layer="1"/>
 <contactref element="R27" pad="2"/>
-<wire x1="10.85" y1="82" x2="10.85" y2="84" width="0" layer="19" extent="1-1"/>
+<wire x1="10.85" y1="84" x2="10.85" y2="82" width="0.254" layer="1"/>
 </signal>
 <signal name="N$3">
