File: controller_pcb_tiny/BlinkyTape Controller.sch (EAGLE design)
At the start: 27 parts, among them CON1 USB_MICROSMT+THRUHULE, Q1 16MHz, U1 MK20D--VFM5, U2 SPI-FLASHSO-8, U3 BRM-2508SMD, U4 74LVC1G17DCK, U6 TPD4S012

Commit message: Rework board to be 29mm, use 0603 package for main cap, add bottom side pad for VUSB, improve +5V routing
Parts:
- removed U$5: POGO_PINSMD, blinkinlabs:POGO_PINSMD
- added RECT_PAD1: TEST_PAD_SMTRECT_PAD, blinkinlabs:TEST_PAD_SMTRECT_PAD
- C7: device adafruit:C-USC0402 -> adafruit:C-USC0603
Connections:
- net GND: no longer U$5.P$1
- net VUSB: now also RECT_PAD1.P$1
Changed lines of the file:
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@@
 <?xml version="1.0" encoding="utf-8"?>
 <!DOCTYPE eagle SYSTEM "eagle.dtd">
-<eagle version="7.1.0">
+<eagle version="7.2.0">
 <drawing>
 <settings>
@@
 </variantdefs>
 <classes>
-<class number="0" name="default" width="0.2032" drill="0.3302">
+<class number="0" name="default" width="0.2032" drill="0.25">
 </class>
 <class number="1" name="power" width="0.3048" drill="0">
@@
 <part name="U$3" library="blinkinlabs" deviceset="POGO_PIN" device="SMD" value="POGO_PINSMD"/>
 <part name="U$4" library="blinkinlabs" deviceset="POGO_PIN" device="SMD" value="POGO_PINSMD"/>
-<part name="U$5" library="blinkinlabs" deviceset="POGO_PIN" device="SMD" value="POGO_PINSMD"/>
 <part name="U$6" library="blinkinlabs" deviceset="POGO_PIN" device="SMD" value="POGO_PINSMD"/>
 <part name="U$7" library="blinkinlabs" deviceset="POGO_PIN" device="SMD" value="POGO_PINSMD"/>
@@
 <part name="GND2" library="supply1" deviceset="GND" device=""/>
 <part name="P+3" library="supply1" deviceset="+5V" device=""/>
-<part name="C7" library="adafruit" deviceset="C-US" device="C0402" value="1uF"/>
+<part name="C7" library="adafruit" deviceset="C-US" device="C0603" value="1uF"/>
+<part name="RECT_PAD1" library="blinkinlabs" deviceset="TEST_PAD_SMT" device="RECT_PAD"/>
 </parts>
 <sheets>
@@
 <instance part="U$3" gate="G$1" x="317.5" y="137.16"/>
 <instance part="U$4" gate="G$1" x="317.5" y="134.62"/>
-<instance part="U$5" gate="G$1" x="335.28" y="139.7" rot="R180"/>
 <instance part="U$6" gate="G$1" x="335.28" y="137.16" rot="R180"/>
 <instance part="U$7" gate="G$1" x="335.28" y="134.62" rot="R180"/>
@@
 </instance>
 <instance part="C7" gate="G$1" x="139.7" y="218.44"/>
+<instance part="RECT_PAD1" gate="G$1" x="317.5" y="86.36" rot="R180"/>
 </instances>
 <busses>
@@
 <pinref part="GND4" gate="1" pin="GND"/>
 <wire x1="127" y1="55.88" x2="127" y2="58.42" width="0.1524" layer="91"/>
-</segment>
-<segment>
-<wire x1="340.36" y1="139.7" x2="347.98" y2="139.7" width="0.1524" layer="91"/>
-<label x="342.9" y="139.7" size="1.778" layer="95"/>
-<pinref part="U$5" gate="G$1" pin="P$1"/>
 </segment>
 <segment>
@@
 <pinref part="D2" gate="G$1" pin="A"/>
 </segment>
-</net>
+<segment>
+<pinref part="RECT_PAD1" gate="G$1" pin="P$1"/>
+<wire x1="322.58" y1="86.36" x2="337.82" y2="86.36" width="0.1524" layer="91"/>
+<label x="327.66" y="86.36" size="1.778" layer="95"/>
+</segment>
+</net>

Commit message: RevA tiny controller
Parts:
- added U$5, U$9: POGO_PINSMD, blinkinlabs:POGO_PINSMD
- U$1: value WS2812B_CONNECTORSTANDARD -> WS2812B_CONNECTOR; device blinkinlabs:WS2812B_CONNECTORSTANDARD -> blinkinlabs:WS2812B_CONNECTOR
Connections:
- net PD5: now also U$5.P$1
- net PD6: now also U$9.P$1
Other:
- note added: "Extra"
Changed lines of the file:
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@@
 <part name="U6" library="blinkinlabs" deviceset="TPD4S012" device=""/>
 <part name="SW1" library="blinkinlabs" deviceset="BUTTON_MOMENTARY" device=""/>
-<part name="U$1" library="blinkinlabs" deviceset="WS2812B_CONNECTOR" device="STANDARD"/>
+<part name="U$1" library="blinkinlabs" deviceset="WS2812B_CONNECTOR" device="" value="WS2812B_CONNECTOR"/>
 <part name="U$2" library="blinkinlabs" deviceset="POGO_PIN" device="SMD" value="POGO_PINSMD"/>
 <part name="U$3" library="blinkinlabs" deviceset="POGO_PIN" device="SMD" value="POGO_PINSMD"/>
@@
 <part name="C7" library="adafruit" deviceset="C-US" device="C0603" value="1uF"/>
 <part name="RECT_PAD1" library="blinkinlabs" deviceset="TEST_PAD_SMT" device="RECT_PAD"/>
+<part name="U$5" library="blinkinlabs" deviceset="POGO_PIN" device="SMD" value="POGO_PINSMD"/>
+<part name="U$9" library="blinkinlabs" deviceset="POGO_PIN" device="SMD" value="POGO_PINSMD"/>
 </parts>
 <sheets>
@@
 <wire x1="274.32" y1="129.54" x2="274.32" y2="45.72" width="0.6096" layer="94"/>
 <text x="203.2" y="119.38" size="5.08" layer="94">IR receiver</text>
+<wire x1="35.56" y1="40.64" x2="124.46" y2="40.64" width="0.6096" layer="94"/>
+<text x="40.64" y="30.48" size="5.08" layer="94">Extra</text>
+<wire x1="35.56" y1="40.64" x2="35.56" y2="5.08" width="0.6096" layer="94"/>
+<wire x1="124.46" y1="40.64" x2="124.46" y2="5.08" width="0.6096" layer="94"/>
+<wire x1="35.56" y1="5.08" x2="124.46" y2="5.08" width="0.6096" layer="94"/>
 </plain>
 <instances>
@@
 <instance part="C7" gate="G$1" x="139.7" y="218.44"/>
 <instance part="RECT_PAD1" gate="G$1" x="317.5" y="86.36" rot="R180"/>
+<instance part="U$5" gate="G$1" x="50.8" y="22.86" rot="R180"/>
+<instance part="U$9" gate="G$1" x="50.8" y="15.24" rot="R180"/>
 </instances>
 <busses>
@@
 <label x="218.44" y="170.18" size="1.778" layer="95"/>
 </segment>
+<segment>
+<pinref part="U$5" gate="G$1" pin="P$1"/>
+<wire x1="55.88" y1="22.86" x2="78.74" y2="22.86" width="0.1524" layer="91"/>
+<label x="63.5" y="22.86" size="1.778" layer="95"/>
+</segment>
 </net>
 <net name="PD7" class="0">
@@
 <label x="218.44" y="167.64" size="1.778" layer="95"/>
 </segment>
-</net>
+<segment>
+<pinref part="U$9" gate="G$1" pin="P$1"/>
+<wire x1="55.88" y1="15.24" x2="78.74" y2="15.24" width="0.1524" layer="91"/>
+<label x="63.5" y="15.24" size="1.778" layer="95"/>
+</segment>
+</net>
